Commit message: Add val3 prototype and improve HW (#6)
Highlights:
- add VAL3 ros2 server, features :
  + custom types and serialization functions
  + read /publish robot state
  + listen for robot command
  + manage cmd FSM (Error -> STOP -> Position -> etc.)
  + implement "real-time" joint position control
- fix HW issues (initialization mostly)

File: staubli_robot_description/r2c/staubli.r2c.xacro (robot description, xacro)
@@ -4,7 +4,8 @@
     <xacro:include filename="$(find staubli_robot_description)/r2c/include/staubli_r2c_joints.xacro" />
     <xacro:include filename="$(find staubli_robot_description)/r2c/include/staubli_r2c_gpios.xacro" />
-    <xacro:macro name="ur_ros2_control" params="
+    <xacro:macro name="staubli_ros2_control" params="
         name
         robot_prefix:=^
+        robot_ip:=^
         robot_model_parameters_file:=^
         initial_positions_file:=^
@@ -23,5 +24,14 @@
             </xacro:if>
             <xacro:unless value="${use_mock_hardware}">
-                <!-- TODO: Implement real hardware interface -->
+                <plugin>staubli_robot_driver/StaubliHardwareInterface</plugin>
+                <param name="robot_ip">${robot_ip}</param>
+                <param name="control_port">56123</param>
+                <param name="diagnostic_port">56124</param>
+                <param name="local_control_port">56123</param>
+                <param name="local_diagnostic_port">56124</param>
+                <param name="num_digital_inputs">${num_digital_inputs}</param>
+                <param name="num_digital_outputs">${num_digital_outputs}</param>
+                <param name="num_analog_inputs">${num_analog_inputs}</param>
+                <param name="num_analog_outputs">${num_analog_outputs}</param>
             </xacro:unless>
         </hardware>
@@ -35,4 +45,5 @@
         />
         <!-- GPIOs -->
+        <!--
         <xacro:r2c_gpios_control_description
             robot_prefix="${robot_prefix}"
@@ -42,4 +53,5 @@
             num_analog_outputs="${num_analog_outputs}"
         />
+        -->
         <!-- GPIOs for Control / Supervision -->
         <!-- TODO -->

File: staubli_robot_description/urdf/staubli.urdf.xacro (robot description, xacro)
@@ -12,4 +12,5 @@
     <xacro:arg name="name" default="staubli"/>
     <xacro:arg name="robot_prefix" default=""/>
+    <xacro:arg name="robot_ip" default="0.0.0.0"/>
     <!-- Set the robot name using the property -->
     <xacro:attribute name="name" value="$(arg name)" />
@@ -59,7 +60,8 @@
     <!-- ROS2 control description -->
     <xacro:include filename="$(find staubli_robot_description)/r2c/staubli.r2c.xacro" />
-    <xacro:ur_ros2_control
+    <xacro:staubli_ros2_control
         name="$(arg name)"
         robot_prefix="$(arg robot_prefix)"
+        robot_ip="$(arg robot_ip)"
         robot_model_parameters_file="$(arg robot_model_parameters_file)"
         initial_positions_file="$(arg initial_positions_file)"
