Commit message: Add acceleration limits (#11)
Highlights:
-  Use real joint limits (i.e., close to robot specs) for TX2-60l
- Set realistic, but downgraded joint limits for moveit 
- Export ACCELERATION interface, without allowing 
- Use ACCELERATION iface to set max acceleration field of joint limiter


* error on switching to acc

File: staubli_robot_description/r2c/include/staubli_r2c_joints.xacro (robot description, xacro)
@@ -3,8 +3,10 @@
     <xacro:macro name="r2c_joints_control_description" params="
         robot_prefix:=^
+        joint_limits_config:=^
         joint_names
         initial_positions
         has_joint_torque_sensor
         has_joint_torque_control
+        include_acceleration_command:=false
     ">
     <xacro:macro name="add_all_rc2_joints" params="robot_prefix:=^ joint_list:=^" >
@@ -13,5 +15,16 @@
             <joint name="${robot_prefix}${joint_name}">
                 <command_interface name="position"/>
-                <command_interface name="velocity"/>
+                <command_interface name="velocity">
+                    <param name="initial_value">0.0</param>
+                </command_interface>
+                <!-- Add acceleration command interface to provide acceleration limits -->
+                <xacro:if value="${include_acceleration_command}">
+                    <xacro:property name="acc_max" value="${joint_limits_config[joint_name]['max_acceleration']}"/>
+                    <command_interface name="acceleration">
+                        <param name="initial_value">0.0</param>
+                        <param name="max">${acc_max}</param>
+                        <param name="min">${-acc_max}</param>
+                    </command_interface>
+                </xacro:if>
                 <xacro:if value="${has_joint_torque_control}">
                     <command_interface name="effort"/>

File: staubli_robot_description/r2c/staubli.r2c.xacro (robot description, xacro)
@@ -9,4 +9,5 @@
         robot_ip:=^
         robot_model_parameters_file:=^
+        joint_limits_parameters_file:=^
         initial_positions_file:=^
         use_mock_hardware:=^
@@ -15,4 +16,5 @@
     <xacro:load_robot_model_config robot_model_config_file="${robot_model_parameters_file}"/>
     <xacro:load_initial_positions_config initial_positions_config_file="${initial_positions_file}"/>
+    <xacro:load_joint_limits_config joint_limits_config_file="${joint_limits_parameters_file}"/>
     <ros2_control name="${name}" type="system">
         <hardware>
@@ -37,4 +39,11 @@
         </hardware>
         <!-- Actuated joints -->
+        <xacro:if value="${use_mock_hardware}">
+            <xacro:property name="include_acceleration_command" value="false"/>
+        </xacro:if>
+        <xacro:unless value="${use_mock_hardware}">
+             <!-- Note: acceleration command interface is ONLY used to set the acceleration limits... -->
+            <xacro:property name="include_acceleration_command" value="true"/>
+        </xacro:unless>
         <xacro:r2c_joints_control_description
             robot_prefix="${robot_prefix}"
@@ -43,4 +52,5 @@
             has_joint_torque_sensor="${has_joint_torque_sensor}"
             has_joint_torque_control="false"
+            include_acceleration_command="${include_acceleration_command}"
         />
         <!-- GPIOs -->

File: staubli_robot_description/urdf/staubli.urdf.xacro (robot description, xacro)
@@ -65,4 +65,5 @@
         robot_ip="$(arg robot_ip)"
         robot_model_parameters_file="$(arg robot_model_parameters_file)"
+        joint_limits_parameters_file="$(arg joint_limits_parameters_file)"
         initial_positions_file="$(arg initial_positions_file)"
         use_mock_hardware="$(arg use_mock_hardware)"
