Commit message: Add (basic) support for gpios (#14)
* move types to separate header

* add GPIO support on HW

File: staubli_robot_description/r2c/include/staubli_r2c_gpios.xacro (robot description, xacro)
@@ -8,10 +8,14 @@
         num_analog_outputs
     ">
-    <xacro:macro name="add_numbered_gpios" params="robot_prefix:=^ interface_name_prefix num_gpios cmd:=false cmd_feedback:= false state:=false current_idx=0" >
+    <xacro:macro name="add_numbered_gpios" params="robot_prefix:=^ interface_name_prefix num_gpios cmd:=false state:=false current_idx=0" >
         <xacro:if value="${current_idx != num_gpios}">
             <xacro:property name="gpio_name" value="${interface_name_prefix}${current_idx}"/>
-            <state_interface name="${gpio_name}">
-                <param name="initial_value">0.0</param>
-            </state_interface>
+            <xacro:if value="${cmd}">
+                <command_interface name="${gpio_name}"/>
+            </xacro:if>
+            <xacro:if value="${state}">
+                <state_interface name="${gpio_name}"/>
+            </xacro:if>
+            <!-- Recursive call -->
             <xacro:add_numbered_gpios
                 robot_prefix="${robot_prefix}"
@@ -19,10 +23,9 @@
                 num_gpios="${num_gpios}"
                 cmd="${cmd}"
-                cmd_feedback="${cmd_feedback}"
                 state="${state}"
                 current_idx="${current_idx + 1}"/>
         </xacro:if>
     </xacro:macro>
-    <gpio name="${robot_prefix}gpios">
+    <gpio name="${robot_prefix}gpio">
         <!-- Digital GPIOs -->
         <xacro:add_numbered_gpios
@@ -32,5 +35,4 @@
             state="true"
             cmd="false"
-            cmd_feedback="false"
         />
         <xacro:add_numbered_gpios
@@ -40,5 +42,4 @@
             state="false"
             cmd="true"
-            cmd_feedback="false"
         />
         <!-- Analog GPIOs -->
@@ -49,5 +50,4 @@
             state="true"
             cmd="false"
-            cmd_feedback="false"
         />
         <xacro:add_numbered_gpios
@@ -57,5 +57,4 @@
             state="false"
             cmd="true"
-            cmd_feedback="false"
         />
     </gpio>

File: staubli_robot_description/r2c/staubli.r2c.xacro (robot description, xacro)
@@ -27,4 +27,5 @@
             <xacro:unless value="${use_mock_hardware}">
                 <plugin>staubli_robot_driver/StaubliHardwareInterface</plugin>
+                <param name="robot_prefix">${robot_prefix}</param>
                 <param name="robot_ip">${robot_ip}</param>
                 <param name="control_port">11000</param>
@@ -54,6 +55,20 @@
             include_acceleration_command="${include_acceleration_command}"
         />
+        <!-- Virtual GPIOs for Control / Supervision -->
+        <gpio name="${robot_prefix}supervision">
+            <!-- Integers -->
+            <state_interface name="operation_mode"/>
+            <state_interface name="operation_mode_status"/>
+            <state_interface name="safety_status"/>
+            <state_interface name="control_sequence_delay"/>
+            <!-- Booleans -->
+            <state_interface name="power_on"/>
+            <state_interface name="motion_possible"/>
+            <state_interface name="in_motion"/>
+            <state_interface name="in_error"/>
+            <state_interface name="estop_pressed"/>
+            <state_interface name="wait_for_ack"/>
+        </gpio>
         <!-- GPIOs -->
-        <!--
         <xacro:r2c_gpios_control_description
             robot_prefix="${robot_prefix}"
@@ -63,7 +78,4 @@
             num_analog_outputs="${num_analog_outputs}"
         />
-        -->
-        <!-- GPIOs for Control / Supervision -->
-        <!-- TODO -->
     </ros2_control>
     </xacro:macro>
